Commit message: Fix Mir file structure

File: sdl_robot_description/urdf/2f140.urdf (robot description, URDF)
Before this commit: robot ur5e_2f140, 13 links, 13 joints
Joints:
- joint ee_tip_joint: parent tool0 -> ur5e_tool0
- joint ur5_ee_link-gripper_base: parent tool0 -> ur5e_tool0

File: sdl_robot_description/urdf/connecting_hardware.urdf.xacro (robot description, xacro)
@@ -24,5 +24,5 @@
   </link>
   <joint name="mir_to_hardware" type="fixed">
-    <parent link="mirbase_footprint"/>
+    <parent link="mir/base_footprint"/>
     <child link="connecting_hardware"/>
     <origin xyz="0.0 0.0 0.0" rpy="0.0 0.0 0.0"/>
@@ -30,5 +30,5 @@
   <joint name="hardware_to_ur" type="fixed">
     <parent link="connecting_hardware"/>
-    <child link="base_link"/>
+    <child link="ur5e_base_link"/>
     <origin xyz="0.325 0.0 0.85" rpy="0.0 0.0 0.0"/>
   </joint>

File: sdl_robot_description/urdf/mir.urdf.xacro (robot description, xacro)
@@ -13,5 +13,5 @@
     <xacro:property name="prefix" value="${tf_prefix_}/" />
   </xacro:unless>
-  <xacro:mir_100 prefix="mir"/>
+  <xacro:mir_100 prefix="mir/"/>
   <!-- <xacro:controller_plugin_gazebo robot_namespace=""/> -->
     <!-- <xacro:diff_controller_plugin_gazebo prefix=""

File: sdl_robot_description/urdf/sdl_robot.urdf.xacro (robot description, xacro)
@@ -5,10 +5,10 @@
   <xacro:include filename="$(find sdl_robot_description)/urdf/common.gazebo.xacro" />
   <!-- mir-->
-  <xacro:include filename="$(find sdl_robot_description)/urdf/mir.urdf.xacro"/>
+  <xacro:include filename="$(find sdl_robot_description)/urdf/mir.urdf.xacro" />
   <!-- connecting hardware -->
   <xacro:include filename="$(find sdl_robot_description)/urdf/connecting_hardware.urdf.xacro" />
   <!-- ur5e arm -->
   <xacro:include filename="$(find ur_e_description)/urdf/ur5e.urdf.xacro" />
-  <xacro:ur5e_robot prefix="" joint_limited="False" />
+  <xacro:ur5e_robot prefix="ur5e_" joint_limited="False" />
 s
   <!-- gripper -->
