Commit message: Commit before branch

File: sdl_robot_description/urdf/ur5e_and_2f140.urdf (robot description, URDF)
Before this commit: robot ur5e_2f140, 24 links, 24 joints
Links:
- link connecting_hardware: geometry collision mesh filename=package://sdl_robot_description/meshes/working_copy_mm.stl scale=0.001 0.001 0.001; visual mesh filename=file:///home/larry/catkin_ws/src/sdl-packages/sdl_robot_des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 scale=0.001 0.001 0.001

Commit message: changed absolute file paths to package paths in urdf

File: sdl_robot_description/urdf/ur5e_and_2f140.urdf (robot description, URDF)
Before this commit: robot ur5e_2f140, 24 links, 24 joints
Links:
- link connecting_hardware: geometry collision mesh filename=package://sdl_robot_description/meshes/working_copy_mm.stl scale=0.001 0.001 0.001; visual mesh filename=package://sdl_robot_description/meshes/working_copy_mm.stl scale=0.001 0.001 0.001
