Commit message: Add mir launch files, create maps, add to README

File: sdl_robot_description/urdf/connecting_hardware.urdf.xacro (robot description, xacro)
@@ -24,5 +24,5 @@
   </link>
   <joint name="mir_to_hardware" type="fixed">
-    <parent link="mir/base_footprint"/>
+    <parent link="base_footprint"/>
     <child link="connecting_hardware"/>
     <origin xyz="0.0 0.0 0.0" rpy="0.0 0.0 0.0"/>

File: sdl_robot_description/urdf/sdl_robot.urdf.xacro (robot description, xacro)
@@ -3,7 +3,7 @@
        name="sdl_robot" >
   <!-- common stuff -->
-  <xacro:include filename="$(find sdl_robot_description)/urdf/common.gazebo.xacro" />
+  <!-- <xacro:include filename="$(find sdl_robot_description)/urdf/common.gazebo.xacro" /> -->
   <!-- mir-->
-  <xacro:include filename="$(find sdl_robot_description)/urdf/mir.urdf.xacro" />
+  <xacro:include filename="$(find mir_description)/urdf/mir.urdf.xacro" />
   <!-- connecting hardware -->
   <xacro:include filename="$(find sdl_robot_description)/urdf/connecting_hardware.urdf.xacro" />
@@ -11,8 +11,7 @@
   <xacro:include filename="$(find ur_description)/urdf/inc/ur5e_macro.xacro" />
   <xacro:ur5e_robot prefix="ur5e_" />
-s
   <!-- gripper -->
   <xacro:include filename="$(find sdl_robot_description)/urdf/2f140.urdf" />
   <!-- camera -->
-  <xacro:include filename="$(find sdl_robot_description)/urdf/camera.urdf.xacro" />
+  <!-- <xacro:include filename="$(find sdl_robot_description)/urdf/camera.urdf.xacro" /> -->
 </robot>

Commit message: changing robot description for customization

File: sdl_robot_description/urdf/connecting_hardware.urdf.xacro (robot description, xacro)
@@ -5,5 +5,5 @@
       <origin xyz="0.1 0 -0.1" rpy="1.57 0 1.57"/>
       <geometry>
-        <mesh filename="package://sdl_robot_description/meshes/working_copy_mm.stl" scale="0.001 0.001 0.001"/>
+        <mesh filename="package://sdl_robot_description/meshes/connection_mockup.stl"/>
       </geometry>
       <material name="LightGrey">
@@ -14,5 +14,5 @@
       <origin xyz="0.1 0 -0.1" rpy="1.57 0 1.57"/>
       <geometry>
-        <mesh filename="package://sdl_robot_description/meshes/working_copy_mm.stl" scale="0.001 0.001 0.001"/>
+        <mesh filename="package://sdl_robot_description/meshes/connection_mockup.stl"/>
       </geometry>
     </collision>

File: sdl_robot_description/urdf/sdl_arm.urdf.xacro (robot description, xacro)
@@ -5,6 +5,7 @@
   <xacro:include filename="$(find sdl_robot_description)/urdf/common.gazebo.xacro" />
   <!-- ur5e arm -->
-  <xacro:include filename="$(find ur_description)/urdf/inc/ur5e_macro.xacro" />
-  <xacro:ur5e_robot prefix="ur5e_" />
+  <xacro:include filename="$(find sdl_robot_description)/urdf/inc/ur5e_macro.xacro" />
+  <xacro:ur5e_robot prefix="ur5e_"
+    transmission_hw_interface="hardware_interface/EffortJointInterface"/>
   <!-- gripper -->
   <xacro:include filename="$(find sdl_robot_description)/urdf/2f140.urdf" />
