Commit message: Working demo

File: sdl_robot_description/urdf/sdl_robot.urdf.xacro (robot description, xacro)
@@ -16,4 +16,13 @@
     <child link="robotiq_arg2f_base_link" />
   </joint>
+  <transmission name="right_outer_knuckle_joint_trans">
+    <type>transmission_interface/SimpleTransmission</type>
+    <joint name="right_outer_knuckle_joint">
+      <hardwareInterface>PositionJointInterface</hardwareInterface>
+    </joint>
+    <actuator name="right_outer_knuckle_joint_motor">
+      <mechanicalReduction>1</mechanicalReduction>
+    </actuator>
+  </transmission>
   <!-- camera -->
   <xacro:include filename="$(find sdl_robot_description)/urdf/camera.urdf.xacro" />
