Commit message: Navigation working

File: sdl_robot_description/urdf/camera.urdf.xacro (robot description, xacro)
@@ -10,5 +10,5 @@
     <parent link="connecting_hardware"/>
     <child link="camera"/>
-    <origin xyz="0 0 .5"/>
+    <origin xyz=".3 0 .5" rpy="0 0 0"/>
   </joint>
   <link name="camera">
@@ -21,5 +21,4 @@
     <visual>
       <geometry>
-        <!-- <box size="0.073000 0.276000 0.072000"/> -->
         <mesh filename="package://sdl_robot_description/urdf/meshes/kinect.dae"/>
       </geometry>

Commit message: Add dependencies to readme

File: sdl_robot_description/urdf/camera.urdf.xacro (robot description, xacro)
@@ -10,5 +10,5 @@
     <parent link="connecting_hardware"/>
     <child link="camera"/>
-    <origin xyz=".3 0 .5" rpy="0 0 0"/>
+    <origin xyz=".5 0 .9" rpy="0 0 0"/>
   </joint>
   <link name="camera">

Commit message: Fix world file, new gripper

File: sdl_robot_description/urdf/camera.urdf.xacro (robot description, xacro)
@@ -21,5 +21,5 @@
     <visual>
       <geometry>
-        <mesh filename="package://sdl_robot_description/urdf/meshes/kinect.dae"/>
+        <mesh filename="package://sdl_robot_description/meshes/kinect.dae"/>
       </geometry>
     </visual>

File: sdl_robot_description/urdf/sdl_robot.urdf.xacro (robot description, xacro)
@@ -12,5 +12,10 @@
   <xacro:ur5e_robot prefix="ur5e_" />
   <!-- gripper -->
-  <xacro:include filename="$(find sdl_robot_description)/urdf/2f140.urdf" />
+  <xacro:include filename="$(find sdl_robot_description)/urdf/robotiq_2f_140_gripper_visualization/urdf/robotiq_arg2f_140_model_macro.xacro" />
+  <xacro:robotiq_arg2f_140 prefix=""/>
+  <joint name="gripper_to_arm" type="fixed" >
+    <parent link="ur5e_tool0" />
+    <child link="robotiq_arg2f_base_link" />
+  </joint>
   <!-- camera -->
   <xacro:include filename="$(find sdl_robot_description)/urdf/camera.urdf.xacro" />

Commit message: Fix file structure

File: sdl_robot_description/urdf/camera.urdf.xacro (robot description, xacro)
@@ -7,10 +7,5 @@
     </inertial>
   </xacro:macro>
-  <joint name="camera_to_hardware" type="fixed">
-    <parent link="connecting_hardware"/>
-    <child link="camera"/>
-    <origin xyz=".5 0 .9" rpy="0 0 0"/>
-  </joint>
-  <link name="camera">
+  <link name="${prefix}camera">
     <xacro:default_inertial mass="1"/>
     <collision>
@@ -26,5 +21,5 @@
   </link>
   <gazebo reference="camera">
-    <sensor name="camera" type="depth">
+    <sensor name="${prefix}camera" type="depth">
       <update_rate>20</update_rate>
       <camera>

File: sdl_robot_description/urdf/connecting_hardware.urdf.xacro (robot description, xacro)
@@ -1,5 +1,5 @@
 <?xml version="1.0"?>
 <robot xmlns:xacro="http://ros.org/wiki/xacro">
-  <link name="connecting_hardware" >
+  <link name="${prefix}connecting_hardware" >
     <visual>
       <origin xyz="0.1 0 -0.1" rpy="1.57 0 1.57"/>
@@ -23,13 +23,3 @@
     </inertial>
   </link>
-  <joint name="mir_to_hardware" type="fixed">
-    <parent link="base_footprint"/>
-    <child link="connecting_hardware"/>
-    <origin xyz="0.0 0.0 0.0" rpy="0.0 0.0 0.0"/>
-  </joint>
-  <joint name="hardware_to_ur" type="fixed">
-    <parent link="connecting_hardware"/>
-    <child link="ur5e_base_link"/>
-    <origin xyz="0.325 0.0 0.85" rpy="0.0 0.0 0.0"/>
-  </joint>
 </robot>

File: sdl_robot_description/urdf/sdl_robot.urdf.xacro (robot description, xacro)
@@ -6,24 +6,58 @@
   <!-- connecting hardware -->
   <xacro:include filename="$(find sdl_robot_description)/urdf/connecting_hardware.urdf.xacro" />
+  <joint name="${prefix}hardware_to_mir" type="fixed">
+    <parent link="${prefix}base_footprint"/>
+    <child link="${prefix}connecting_hardware"/>
+    <origin xyz="0.0 0.0 0.0" rpy="0.0 0.0 0.0"/>
+  </joint>
   <!-- ur5e arm -->
   <xacro:include filename="$(find sdl_robot_description)/urdf/inc/ur5e_macro.xacro" />
-  <xacro:ur5e_robot prefix="ur5e_" />
+  <xacro:ur5e_robot prefix="${prefix}ur5e_" />
+  <joint name="${prefix}ur_to_hardware" type="fixed">
+    <parent link="${prefix}connecting_hardware"/>
+    <child link="${prefix}ur5e_base_link"/>
+    <origin xyz="0.325 0.0 0.85" rpy="0.0 0.0 0.0"/>
+  </joint>
   <!-- gripper -->
   <xacro:include filename="$(find robotiq_2f_140_gripper_visualization)/urdf/robotiq_arg2f_140_model_macro.xacro" />
   <xacro:robotiq_arg2f_140 prefix=""/>
-  <joint name="gripper_to_arm" type="fixed" >
-    <parent link="ur5e_tool0" />
-    <child link="robotiq_arg2f_base_link" />
+  <joint name="${prefix}gripper_to_ur" type="fixed" >
+    <parent link="${prefix}ur5e_tool0" />
+    <child link="${prefix}robotiq_arg2f_base_link" />
   </joint>
-  <transmission name="right_outer_knuckle_joint_trans">
-    <type>transmission_interface/SimpleTransmission</type>
-    <joint name="right_outer_knuckle_joint">
-      <hardwareInterface>PositionJointInterface</hardwareInterface>
-    </joint>
-    <actuator name="right_outer_knuckle_joint_motor">
-      <mechanicalReduction>1</mechanicalReduction>
-    </actuator>
-  </transmission>
+  <gazebo>
+      <!-- loading plugin: mimic joints works in gazebo now-->
+    <plugin filename="libroboticsgroup_upatras_gazebo_mimic_joint_plugin.so" name="${prefix}mimic_robotiq_140_4">
+        <joint>${prefix}finger_joint</joint>
+        <mimicJoint>${prefix}right_outer_knuckle_joint</mimicJoint>
+        <multiplier>-1.0</multiplier>
+    </plugin>
+    <plugin filename="libroboticsgroup_upatras_gazebo_mimic_joint_plugin.so" name="${prefix}mimic_robotiq_140_2">
+        <joint>${prefix}finger_joint</joint>
+        <mimicJoint>${prefix}left_inner_finger_joint</mimicJoint>
+        <multiplier>1.0</multiplier>
+    </plugin>
+    <plugin filename="libroboticsgroup_upatras_gazebo_mimic_joint_plugin.so" name="${prefix}mimic_robotiq_140_5">
+        <joint>${prefix}finger_joint</joint>
+        <mimicJoint>${prefix}right_inner_finger_joint</mimicJoint>
+        <multiplier>1.0</multiplier>
+    </plugin>
+    <plugin filename="libroboticsgroup_upatras_gazebo_mimic_joint_plugin.so" name="${prefix}mimic_robotiq_140_3">
+        <joint>${prefix}finger_joint</joint>
+        <mimicJoint>${prefix}left_inner_knuckle_joint</mimicJoint>
+        <multiplier>-1.0</multiplier>
+    </plugin>
+    <plugin filename="libroboticsgroup_upatras_gazebo_mimic_joint_plugin.so" name="${prefix}mimic_robotiq_140_5">
+        <joint>${prefix}finger_joint</joint>
+        <mimicJoint>${prefix}right_inner_knuckle_joint</mimicJoint>
+        <multiplier>-1.0</multiplier>
+    </plugin>
+  </gazebo>
   <!-- camera -->
   <xacro:include filename="$(find sdl_robot_description)/urdf/camera.urdf.xacro" />
+  <joint name="${prefix}camera_to_hardware" type="fixed">
+    <parent link="${prefix}connecting_hardware"/>
+    <child link="${prefix}camera"/>
+    <origin xyz=".5 0 .9" rpy="0 0 0"/>
+  </joint>
 </robot>
