Commit message: Fix readme

File: sdl_robot_description/urdf/2f140.urdf.xacro (robot description, xacro)
@@ -1,29 +1,6 @@
 <?xml version="1.0"?>
-<robot xmlns:xacro="http://ros.org/wiki/xacro"
-       name="sdl_robot" >
-  <!-- mir-->
-  <xacro:include filename="$(find mir_description)/urdf/mir.urdf.xacro" />
-  <!-- connecting hardware -->
-  <xacro:include filename="$(find sdl_robot_description)/urdf/connecting_hardware.urdf.xacro" />
-  <joint name="${prefix}hardware_to_mir" type="fixed">
-    <parent link="${prefix}base_footprint"/>
-    <child link="${prefix}connecting_hardware"/>
-    <origin xyz="0.0 0.0 0.0" rpy="0.0 0.0 0.0"/>
-  </joint>
-  <!-- ur5e arm -->
-  <xacro:include filename="$(find sdl_robot_description)/urdf/inc/ur5e_macro.xacro" />
-  <xacro:ur5e_robot prefix="${prefix}ur5e_" />
-  <joint name="${prefix}ur_to_hardware" type="fixed">
-    <parent link="${prefix}connecting_hardware"/>
-    <child link="${prefix}ur5e_base_link"/>
-    <origin xyz="0.325 0.0 0.85" rpy="0.0 0.0 0.0"/>
-  </joint>
-  <!-- gripper -->
+<robot xmlns:xacro="http://ros.org/wiki/xacro" >
   <xacro:include filename="$(find robotiq_2f_140_gripper_visualization)/urdf/robotiq_arg2f_140_model_macro.xacro" />
-  <xacro:robotiq_arg2f_140 prefix=""/>
-  <joint name="${prefix}gripper_to_ur" type="fixed" >
-    <parent link="${prefix}ur5e_tool0" />
-    <child link="${prefix}robotiq_arg2f_base_link" />
-  </joint>
+  <xacro:robotiq_arg2f_140 prefix="${prefix}"/>
   <gazebo>
       <!-- loading plugin: mimic joints works in gazebo now-->
@@ -54,10 +31,19 @@
     </plugin>
   </gazebo>
-  <!-- camera -->
-  <xacro:include filename="$(find sdl_robot_description)/urdf/camera.urdf.xacro" />
-  <joint name="${prefix}camera_to_hardware" type="fixed">
-    <parent link="${prefix}connecting_hardware"/>
-    <child link="${prefix}camera"/>
-    <origin xyz=".5 0 .9" rpy="0 0 0"/>
-  </joint>
+  <gazebo reference="right_inner_finger">
+    <implicitSpringDamper>1</implicitSpringDamper>
+    <kp>1000000.0</kp>
+    <kd>1.0</kd>
+    <mu1>1.0</mu1>
+    <mu2>1.0</mu2>
+    <minDepth>0.001</minDepth>
+  </gazebo>
+  <gazebo reference="left_inner_finger">
+    <implicitSpringDamper>1</implicitSpringDamper>
+    <kp>1000000.0</kp>
+    <kd>1.0</kd>
+    <mu1>1.0</mu1>
+    <mu2>1.0</mu2>
+    <minDepth>0.001</minDepth>
+  </gazebo>
 </robot>
